Commit message: Increased caster wheel size and reduced lidar weight to make robot balance in simulations

File: src/arsenal_navigator/description/robot_core.xacro (robot description, xacro)
@@ -4,12 +4,12 @@
     <xacro:property name="chassis_radius" value="0.049"/>
     <xacro:property name="chassis_height" value="0.453"/>
-    <xacro:property name="wheel_radius" value="0.031"/>
-    <xacro:property name="wheel_thickness" value="0.015"/>
+    <xacro:property name="wheel_radius" value="0.035"/>
+    <xacro:property name="wheel_thickness" value="0.025"/>
     <xacro:property name="wheel_offset_y" value="0.06"/>
-    <xacro:property name="wheel_offset_z" value="-0.011"/>
+    <xacro:property name="wheel_offset_z" value="-0.015"/>
     <xacro:property name="wheel_offset_x" value="0.065"/>
     <xacro:property name="wheel_mass" value="0.03"/>
-    <xacro:property name="caster_wheel_mass" value="0.01"/>
-    <xacro:property name="caster_wheel_radius" value="0.01"/>
+    <xacro:property name="caster_wheel_mass" value="0.02"/>
+    <xacro:property name="caster_wheel_radius" value="0.015"/>
     <xacro:property name="caster_wheel_offset_x" value="0.049"/>
     <xacro:property name="caster_wheel_offset_z" value="${wheel_offset_z - wheel_radius + caster_wheel_radius}"/>
@@ -26,6 +26,8 @@
         <color rgba="0 0 0 1"/>
     </material>
+    <!--Base Link-->
     <link name="base_link">
     </link>
+    <!--Base Footprint Link-->
     <link name="base_footprint">
     </link>
@@ -56,5 +58,5 @@
         </collision>
         <xacro:inertial_cylinder mass="1.0" length="${chassis_height}" radius="${chassis_radius}">
-            <origin xyz="0.049 0 ${chassis_height/2}" rpy="0 0 0"/>
+            <origin xyz="0.049 0 ${chassis_height/10}" rpy="0 0 0"/>
         </xacro:inertial_cylinder>
     </link>
