Commit message: updated lidar description

File: src/arsenal_navigator/description/lidar.xacro (robot description, xacro)
@@ -17,5 +17,5 @@
         </visual>
         <collision>
-            <origin xyz="0.049 0 ${chassis_height/2}"/>
+            <origin xyz="0 0 0"/>
             <geometry>
                 <cylinder radius="${chassis_radius}" length="${lidar_height}"/>
@@ -23,6 +23,33 @@
         </collision>
         <xacro:inertial_cylinder mass="0.05" length="${lidar_height}" radius="${chassis_radius}">
-            <origin xyz="0.049 0 ${chassis_height/2}" rpy="0 0 0"/>
+            <origin xyz="0 0 0" rpy="0 0 0"/>
         </xacro:inertial_cylinder>
     </link>
+    <gazebo reference="laser_frame">
+        <sensor name="laser" type="ray">
+            <pose> 0 0 0 0 0 0 </pose>
+            <visualize>true</visualize>
+            <update_rate>15</update_rate>
+            <ray>
+                <scan>
+                    <horizontal>
+                        <samples>360</samples>
+                        <min_angle>-3.14</min_angle>
+                        <max_angle>3.14</max_angle>
+                    </horizontal>
+                </scan>
+                <range>
+                    <min>0.3</min>
+                    <max>8</max>
+                </range>
+            </ray>
+            <plugin name="laser_controller" filename="libgazebo_ros_ray_sensor.so">
+                <ros>
+                    <argument>~/out:=scan</argument>
+                </ros>
+                <output_type>sensor_msgs/LaserScan</output_type>
+                <frame_name>laser_frame</frame_name>
+            </plugin>
+        </sensor>
+    </gazebo>
 </robot>
