Commit message: added robot description files

File: src/arsenal_navigator/description/arsenal_robot_description.urdf.xacro (robot description, xacro)
@@ -1,6 +1,16 @@
 <?xml version="1.0"?>
-<robot name="arsenal_robot" xmlns:xacro="http://ros.org/wiki/xacro">
+<robot xmlns:xacro="http://www.ros.org/wiki/xacro"  name="robot">
     <xacro:arg name="use_ros2_control" default="true"/>
     <xacro:arg name="sim_mode" default="false"/>
-    <xacro:include filename="robot_core.xacro"/>
+    <xacro:include filename="robot_core.xacro" />
+    <xacro:if value="$(arg use_ros2_control)">
+        <xacro:include filename="ros2_control.xacro" />
+    </xacro:if>
+    <xacro:unless value="$(arg use_ros2_control)">
+        <xacro:include filename="gazebo_control.xacro" />
+    </xacro:unless>
+    <xacro:include filename="lidar.xacro" />
+    <!--<xacro:include filename="camera.xacro" />-->
+    <!-- <xacro:include filename="depth_camera.xacro" /> -->
+   <!-- <xacro:include filename="face.xacro" />-->
 </robot>

File: src/arsenal_navigator/description/robot_core.xacro (robot description, xacro)
@@ -28,4 +28,11 @@
     <link name="base_link">
     </link>
+    <link name="base_footprint">
+    </link>
+    <joint name="base_joint" type="fixed">
+        <parent link="base_link"/>
+        <child link="base_footprint"/>
+        <origin xyz="0.0 0.0 0.0" rpy="0 0 0"/>
+    </joint>
     <!--Chassis Link-->
     <joint name="chassis_joint" type="fixed">

Commit message: updated robot description

File: src/arsenal_navigator/description/arsenal_robot_description.urdf.xacro (robot description, xacro)
@@ -2,5 +2,5 @@
 <robot xmlns:xacro="http://www.ros.org/wiki/xacro"  name="robot">
     <xacro:arg name="use_ros2_control" default="true"/>
-    <xacro:arg name="sim_mode" default="false"/>
+    <xacro:arg name="sim_mode" default="true"/>
     <xacro:arg name="sim_lidar" default="true"/>
     <xacro:include filename="robot_core.xacro" />

File: src/arsenal_navigator/description/gazebo_control.xacro (robot description, xacro)
@@ -9,6 +9,6 @@
             <wheel_diameter>0.062</wheel_diameter>
             <!-- Limits -->
-            <max_wheel_torque>200</max_wheel_torque>
-            <max_wheel_acceleration>10.0</max_wheel_acceleration>
+            <max_wheel_torque>20</max_wheel_torque>
+            <max_wheel_acceleration>5.0</max_wheel_acceleration>
             <!-- Output -->
             <odometry_frame>odom</odometry_frame>

File: src/arsenal_navigator/description/lidar_sim.xacro (robot description, xacro)
@@ -17,5 +17,5 @@
         </visual>
         <collision>
-            <origin xyz="0.049 0 ${chassis_height/2}"/>
+            <origin xyz="0 0 0"/>
             <geometry>
                 <cylinder radius="${chassis_radius}" length="${lidar_height}"/>
@@ -23,5 +23,5 @@
         </collision>
         <xacro:inertial_cylinder mass="0.05" length="${lidar_height}" radius="${chassis_radius}">
-            <origin xyz="0.049 0 ${chassis_height/2}" rpy="0 0 0"/>
+            <origin xyz="0 0 0" rpy="0 0 0"/>
         </xacro:inertial_cylinder>
     </link>
@@ -30,5 +30,5 @@
             <pose> 0 0 0 0 0 0 </pose>
             <visualize>true</visualize>
-            <update_rate>10</update_rate>
+            <update_rate>15</update_rate>
             <ray>
                 <scan>
@@ -44,5 +44,5 @@
                 </range>
             </ray>
-            <!--<plugin name="laser_controller" filename="libgazebo_ros_ray_sensor.so">
+            <plugin name="laser_controller" filename="libgazebo_ros_ray_sensor.so">
                 <ros>
                     <argument>~/out:=scan</argument>
@@ -50,5 +50,5 @@
                 <output_type>sensor_msgs/LaserScan</output_type>
                 <frame_name>laser_frame</frame_name>
-            </plugin>-->
+            </plugin>
         </sensor>
     </gazebo>

File: src/arsenal_navigator/description/robot_core.xacro (robot description, xacro)
@@ -4,13 +4,13 @@
     <xacro:property name="chassis_radius" value="0.049"/>
     <xacro:property name="chassis_height" value="0.453"/>
-    <xacro:property name="wheel_radius" value="0.035"/>
-    <xacro:property name="wheel_thickness" value="0.025"/>
+    <xacro:property name="wheel_radius" value="0.03"/>
+    <xacro:property name="wheel_thickness" value="0.015"/>
     <xacro:property name="wheel_offset_y" value="0.06"/>
-    <xacro:property name="wheel_offset_z" value="-0.015"/>
+    <xacro:property name="wheel_offset_z" value="-0.016"/>
     <xacro:property name="wheel_offset_x" value="0.065"/>
-    <xacro:property name="wheel_mass" value="0.03"/>
+    <xacro:property name="wheel_mass" value="0.05"/>
     <xacro:property name="caster_wheel_mass" value="0.02"/>
     <xacro:property name="caster_wheel_radius" value="0.015"/>
-    <xacro:property name="caster_wheel_offset_x" value="0.049"/>
+    <xacro:property name="caster_wheel_offset_x" value="0.07"/>
     <xacro:property name="caster_wheel_offset_z" value="${wheel_offset_z - wheel_radius + caster_wheel_radius}"/>
     <material name="white">
@@ -58,5 +58,5 @@
         </collision>
         <xacro:inertial_cylinder mass="1.0" length="${chassis_height}" radius="${chassis_radius}">
-            <origin xyz="0.049 0 ${chassis_height/10}" rpy="0 0 0"/>
+            <origin xyz="0.049 0 ${chassis_height/2}" rpy="0 0 0"/>
         </xacro:inertial_cylinder>
     </link>
@@ -78,7 +78,20 @@
             </geometry>
         </visual>
-        <collision>
-            <geometry>
-                <cylinder radius="${wheel_radius}" length="${wheel_thickness}"/>
+        <surface>
+            <friction>
+            <ode>
+                <mu>1.0</mu>
+                <mu2>1.0</mu2>
+            </ode>
+            </friction>
+            <contact>
+            <ode>
+                <min_depth>0.08</min_depth>
+            </ode>
+            </contact>
+        </surface>
+        <collision>
+            <geometry>
+                <sphere radius="${wheel_radius}"/>
             </geometry>
         </collision>
@@ -104,7 +117,20 @@
             </geometry>
         </visual>
-        <collision>
-            <geometry>
-                <cylinder radius="${wheel_radius}" length="${wheel_thickness}"/>
+        <surface>
+            <friction>
+                <ode>
+                    <mu>1.0</mu>
+                    <mu2>1.0</mu2>
+                </ode>
+            </friction>
+            <contact>
+                <ode>
+                    <min_depth>0.08</min_depth>
+                </ode>
+            </contact>
+        </surface>
+        <collision>
+            <geometry>
+                <sphere radius="${wheel_radius}" />
             </geometry>
         </collision>
@@ -120,5 +146,5 @@
         <parent link="chassis"/>
         <child link="front_caster_wheel"/>
-        <origin xyz="0 0 0"/>
+        <origin xyz="-${caster_wheel_offset_x} 0 0"/>
     </joint>
     <link name="front_caster_wheel">
@@ -134,4 +160,9 @@
             </geometry>
         </collision>
+        <contact>
+            <ode>
+                <min_depth>0.1</min_depth>
+            </ode>
+        </contact>
         <xacro:inertial_sphere mass="${caster_wheel_mass}" radius="${caster_wheel_radius}">
             <origin xyz="0 0 0" rpy="0 0 0"/>
@@ -147,5 +178,5 @@
         <parent link="chassis"/>
         <child link="back_caster_wheel"/>
-        <origin xyz="${(2*chassis_radius)} 0 0"/>
+        <origin xyz="${(2*chassis_radius) + caster_wheel_offset_x} 0 0"/>
     </joint>
     <link name="back_caster_wheel">
@@ -156,4 +187,9 @@
             <material name="white"/>
         </visual>
+        <contact>
+            <ode>
+                <min_depth>0.1</min_depth>
+            </ode>
+        </contact>
         <collision>
             <geometry>

File: src/arsenal_navigator/description/ros2_control.xacro (robot description, xacro)
@@ -15,6 +15,6 @@
             <joint name="left_wheel_joint">
                 <command_interface name="velocity">
-                    <param name="min">-10</param>
-                    <param name="max">10</param>
+                    <param name="min">-2</param>
+                    <param name="max">2</param>
                 </command_interface>
                 <state_interface name="position"/>
@@ -23,6 +23,6 @@
             <joint name="right_wheel_joint">
                 <command_interface name="velocity">
-                    <param name="min">-10</param>
-                    <param name="max">10</param>
+                    <param name="min">-2</param>
+                    <param name="max">2</param>
                 </command_interface>
                 <state_interface name="position"/>
@@ -38,6 +38,6 @@
             <joint name="left_wheel_joint">
                 <command_interface name="velocity">
-                    <param name="min">-10</param>
-                    <param name="max">10</param>
+                    <param name="min">-2</param>
+                    <param name="max">2</param>
                 </command_interface>
                 <state_interface name="velocity"/>
@@ -46,6 +46,6 @@
             <joint name="right_wheel_joint">
                 <command_interface name="velocity">
-                    <param name="min">-10</param>
-                    <param name="max">10</param>
+                    <param name="min">-2</param>
+                    <param name="max">2</param>
                 </command_interface>
                 <state_interface name="velocity"/>

Commit message: final

File: src/arsenal_navigator/description/arsenal_robot_description.urdf.xacro (robot description, xacro)
@@ -12,4 +12,6 @@
     </xacro:if>
     <xacro:include filename="lidar.xacro" />
-    <xacro:include filename="camera.xacro" />
+    <!--<xacro:include filename="camera.xacro" />-->
+    <!-- <xacro:include filename="depth_camera.xacro" /> -->
+   <!-- <xacro:include filename="face.xacro" />-->
 </robot>

File: src/arsenal_navigator/description/lidar.xacro (robot description, xacro)
@@ -46,5 +46,5 @@
             <plugin name="laser_controller" filename="libgazebo_ros_ray_sensor.so">
                 <ros>
-                    <argument>~/out:=scan</argument>
+                    <argument>--ros-args --remap /laser_controller/out:=scan</argument>
                 </ros>
                 <output_type>sensor_msgs/LaserScan</output_type>

File: src/arsenal_navigator/description/robot_core.xacro (robot description, xacro)
@@ -4,5 +4,5 @@
     <xacro:property name="chassis_radius" value="0.049"/>
     <xacro:property name="chassis_height" value="0.453"/>
-    <xacro:property name="wheel_radius" value="0.03"/>
+    <xacro:property name="wheel_radius" value="0.0335"/>
     <xacro:property name="wheel_thickness" value="0.015"/>
     <xacro:property name="wheel_offset_y" value="0.06"/>

File: src/arsenal_navigator/description/ros2_control.xacro (robot description, xacro)
@@ -12,6 +12,6 @@
             <joint name="left_wheel_joint">
                 <command_interface name="velocity">
-                    <param name="min">-5</param>
-                    <param name="max">5</param>
+                    <param name="min">-10</param>
+                    <param name="max">10</param>
                 </command_interface>
                 <state_interface name="position"/>
@@ -20,6 +20,6 @@
             <joint name="right_wheel_joint">
                 <command_interface name="velocity">
-                    <param name="min">-5</param>
-                    <param name="max">5</param>
+                    <param name="min">-10</param>
+                    <param name="max">10</param>
                 </command_interface>
                 <state_interface name="position"/>
